Commit message: Update mpu6050 urdf and bringup files

File: mpu6050_demo_description/urdf/mpu6050.urdf.xacro (robot description, xacro)
@@ -1,16 +1,23 @@
 <?xml version="1.0" ?>
 <robot name="mpu6050_sensor" xmlns:xacro="http://ros.org/wiki/xacro">
+    <!-- World link -->
+    <link name="world"/>
     <!-- Base link -->
     <link name="base_link"/>
+    <joint name="world_joint" type="fixed">
+        <parent link="world"/>
+        <child link="base_link"/>
+        <origin xyz="0 0 0.5" rpy="0 0 0"/>
+    </joint>
     <!-- Imu link  -->
     <link name="imu_link">
       <visual name="imu_visual">
         <geometry>
-        <!-- <mesh filename="package://lidarbot_description/meshes/MPU6050.dae"/> -->
-          <mesh filename="package://lidarbot_description/meshes/MPU6050.dae" scale="100 100 100"/>
+          <mesh filename="package://mpu6050_demo_description/meshes/MPU6050.dae" scale="100 100 100"/>
         </geometry>
       </visual>
     </link>
-    <joint name="imu_joint" type="fixed">
+    <joint name="imu_joint" type="floating">
+<!-- <joint name="imu_joint" type="fixed"> -->
         <parent link="base_link"/>
         <child link="imu_link"/>
